Commit message: model color fixed

File: osiris_bot/urdf/mybot.xacro (robot description, xacro)
@@ -24,4 +24,5 @@
                 <box size=".4 .2 .1" />
             </geometry>
+            <material name="orange" />
         </visual>
     </link>
@@ -41,4 +42,5 @@
                 <cylinder radius="0.1" length="0.05" />
             </geometry>
+            <material name="blue" />
         </visual>
         <inertial>
@@ -65,4 +67,5 @@
                 <cylinder radius="0.1" length="0.05" />
             </geometry>
+            <material name="blue" />
         </visual>
         <inertial>
@@ -110,4 +113,5 @@
                 <cylinder radius="0.1" length="0.05" />
             </geometry>
+            <material name="blue" />
         </visual>
         <inertial>
@@ -134,4 +138,5 @@
                 <cylinder radius="0.1" length="0.05" />
             </geometry>
+            <material name="blue" />
         </visual>
         <inertial>
@@ -235,4 +240,5 @@
                 <cylinder length="0.015" radius="0.01" />
             </geometry>
+            <material name="red" />
         </visual>
         <collision>
